File: oresat-design-blocks/at86rf215-design-block/at86rf215-design-block-sch-radio.kicad_sch (KiCad schematic)
At the start: 45 parts, among them J1 SMA, J10 Conn_01x08, J11 Conn_01x05, J12 Conn_01x08, J2 USB4105-GF-A, J3 Conn_01x06, J6 Conn_01x06, J9 Screw_Terminal_01x02, SW1 RESET, U1 AT86RF215, U2 LP2985AIM5-1.8_NOPB, X1 TXETALSANF-26.000000

Commit message: Last of the GPS card cleanup
Better plains in the RF section, lots of shortening and straitening, cleaned up all ERC and DRCs.
Connections:
- net at C13.2: now also J2.SH (SHIELD); no longer J2.S1 (SHIELD)
Changed lines of the file:
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@@
 	(title_block
 		(title "OreSat AT86RF215 Evaluation Board")
-		(date "2025-12-16")
-		(rev "1.0")
+		(date "2026-05-27")
+		(rev "1.1")
 		(company "Portland State Aerospace Society")
 	)
@@
 		(dnp no)
 		(property "Reference" "J2"
-			(at 64.77 43.688 0)
+			(at 72.39 43.815 0)
 			(show_name no)
 			(do_not_autoplace no)
@@
 			)
 		)
-		(property "Description" "USB-C (USB TYPE-C) USB 2.0 Receptacle Connector 24 (16+8 Dummy) Position Surface Mount, Right Angle; Through Hole"
+		(property "Description" "USB 2.0-only 16P Type-C Receptacle connector"
 			(at 72.39 66.04 0)
 			(hide yes)
@@
 		(pin "A8"
 		)
-		(pin "S1"
+		(pin "SH"
 		)
 		(pin "A1"
