File: oresat-design-blocks/at86rf215-design-block/at86rf215-design-block.kicad_pcb (KiCad board)
At the start: 4 copper layers, 61.3 x 44.1 mm, 80 parts, among them J1 SMA, J10 Conn_01x08, J11 Conn_01x05, J12 Conn_01x08, J2 USB4105-GF-A, J3 Conn_01x06, J4 SMA, J6 Conn_01x06, J7 SMA, J8 SMA, J9 Screw_Terminal_01x02, SW1 RESET, U1 AT86RF215, U2 LP2985AIM5-1.8_NOPB, U3 2450FB15A050E, U4 NCS2-62+, U5 QPC1022, X1 TXETALSANF-26.000000

Commit message: Last of the GPS card cleanup
Better plains in the RF section, lots of shortening and straitening, cleaned up all ERC and DRCs.
Connections:
- J2 pad S1: Net-(J2-SHIELD) -> (no net)
Changed lines of the file:
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@@
 	(title_block
 		(title "AT86RF215 Breakout")
-		(date "2025-12-22")
-		(rev "1.0")
+		(date "2026-05-27")
+		(rev "1.1")
 		(company "Portland State Aerospace Society")
 	)
@@
 			)
 		)
-		(property "Description" "USB-C (USB TYPE-C) USB 2.0 Receptacle Connector 24 (16+8 Dummy) Position Surface Mount, Right Angle; Through Hole"
+		(property "Description" "USB 2.0-only 16P Type-C Receptacle connector"
 			(at 0 0 180)
 			(unlocked yes)
@@
 			(unit
 				(name "A")
-				(pins "S1" "B1" "B12" "A1" "A12" "A9" "B4" "B9" "A4" "A5" "B5" "A7" "B7"
+				(pins "SH" "B1" "B12" "A1" "A12" "A9" "B4" "B9" "A4" "A5" "B5" "A7" "B7"
 					"A6" "B6" "A8" "B8"
 				)
@@
 			(layers "*.Cu" "*.Mask")
 			(remove_unused_layers no)
-			(net "Net-(J2-SHIELD)")
-			(pinfunction "SHIELD_S1")
-			(pintype "passive")
 		)
 		(pad "S1" thru_hole oval
@@
 			(layers "*.Cu" "*.Mask")
 			(remove_unused_layers no)
-			(net "Net-(J2-SHIELD)")
-			(pinfunction "SHIELD_S1")
-			(pintype "passive")
 		)
 		(pad "S1" thru_hole oval
@@
 			(layers "*.Cu" "*.Mask")
 			(remove_unused_layers no)
-			(net "Net-(J2-SHIELD)")
-			(pinfunction "SHIELD_S1")
-			(pintype "passive")
 		)
 		(pad "S1" thru_hole oval
@@
 			(layers "*.Cu" "*.Mask")
 			(remove_unused_layers no)
-			(net "Net-(J2-SHIELD)")
-			(pinfunction "SHIELD_S1")
-			(pintype "passive")
 		)
 		(embedded_fonts no)
